Commit message: Added virtual links for closed chains and corner collision links

File: urdf/robogami.urdf (robot description, URDF)
Before this commit: robot Robogami, 14 links, 13 joints
Links:
- added link leg1lowerLeftConner; collision sphere radius=0.001; visual sphere radius=0.001
- added link leg1lowerRightConner; collision sphere radius=0.001; visual sphere radius=0.001
- added link leg1topLeftConner; collision sphere radius=0.001; visual sphere radius=0.001
- added link leg1topRightConner; collision sphere radius=0.001; visual sphere radius=0.001
- added link leg2TopMove
- added link leg2lowerLeftConner; collision sphere radius=0.001; visual sphere radius=0.001
- added link leg2lowerRightConner; collision sphere radius=0.001; visual sphere radius=0.001
- added link leg2topLeftConner; collision sphere radius=0.001; visual sphere radius=0.001
- added link leg2topRightConner; collision sphere radius=0.001; visual sphere radius=0.001
- added link leg3TopMove
- added link leg3lowerLeftConner; collision sphere radius=0.001; visual sphere radius=0.001
- added link leg3lowerRightConner; collision sphere radius=0.001; visual sphere radius=0.001
- added link leg3topLeftConner; collision sphere radius=0.001; visual sphere radius=0.001
- added link leg3topRightConner; collision sphere radius=0.001; visual sphere radius=0.001
Joints:
- added joint l2TopMove: type revolute, parent leg2top, child leg2TopMove, origin xyz=0.059 0 0 rpy=0 0 0, axis 0 1 0, limit lower=0 upper=1.56 effort=1 velocity=1
- added joint l3TopMove: type revolute, parent leg3top, child leg3TopMove, origin xyz=0.059 0 0 rpy=0 0 0, axis 0 1 0, limit lower=0 upper=1.56 effort=1 velocity=1
- added joint leg1lowerLeftConner_joint: type fixed, parent leg1, child leg1lowerLeftConner, origin xyz=-0.038442059036156634 -0.0245 0 rpy=0 0 0
- added joint leg1lowerRightConner_joint: type fixed, parent leg1, child leg1lowerRightConner, origin xyz=-0.038442059036156634 0.0245 0 rpy=0 0 0
- added joint leg1topLeftConner_joint: type fixed, parent leg1top, child leg1topLeftConner, origin xyz=0.02055794096384336 -0.0245 0 rpy=0 0 0
- added joint leg1topRightConner_joint: type fixed, parent leg1top, child leg1topRightConner, origin xyz=0.02055794096384336 0.0245 0 rpy=0 0 0
- added joint leg2lowerLeftConner_joint: type fixed, parent leg2, child leg2lowerLeftConner, origin xyz=-0.038442059036156634 -0.0245 0 rpy=0 0 0
- added joint leg2lowerRightConner_joint: type fixed, parent leg2, child leg2lowerRightConner, origin xyz=-0.038442059036156634 0.0245 0 rpy=0 0 0
- added joint leg2topLeftConner_joint: type fixed, parent leg2top, child leg2topLeftConner, origin xyz=0.02055794096384336 -0.0245 0 rpy=0 0 0
- added joint leg2topRightConner_joint: type fixed, parent leg2top, child leg2topRightConner, origin xyz=0.02055794096384336 0.0245 0 rpy=0 0 0
- added joint leg3lowerLeftConner_joint: type fixed, parent leg3, child leg3lowerLeftConner, origin xyz=-0.038442059036156634 -0.0245 0 rpy=0 0 0
- added joint leg3lowerRightConner_joint: type fixed, parent leg3, child leg3lowerRightConner, origin xyz=-0.038442059036156634 0.0245 0 rpy=0 0 0
- added joint leg3topLeftConner_joint: type fixed, parent leg3top, child leg3topLeftConner, origin xyz=0.02055794096384336 -0.0245 0 rpy=0 0 0
- added joint leg3topRightConner_joint: type fixed, parent leg3top, child leg3topRightConner, origin xyz=0.02055794096384336 0.0245 0 rpy=0 0 0

Commit message: Finalized contact surface file generation

File: urdf/robogami.urdf (robot description, URDF)
Before this commit: robot Robogami, 28 links, 27 joints
Links:
- added link topleg2
- added link topleg3
Joints:
- added joint topleg2: type fixed, parent top, child topleg2, origin xyz=-0.08443747686898277 -0.04875 0 rpy=0 1.5707963267948966 -2.0943951023931953
- added joint topleg3: type fixed, parent top, child topleg3, origin xyz=-0.08443747686898277 0.04875 0 rpy=0 1.5707963267948966 2.0943951023931953
- joint l2TopMove: limit lower=0 upper=1.56 effort=1 velocity=1 -> lower=-1.56 upper=1.56 effort=1 velocity=1; origin xyz=0.059 0 0 rpy=0 0 0 -> xyz=0.059 0 0 rpy=0 -1.5707963267948966 0
- joint l3TopMove: limit lower=0 upper=1.56 effort=1 velocity=1 -> lower=-1.56 upper=1.56 effort=1 velocity=1; origin xyz=0.059 0 0 rpy=0 0 0 -> xyz=0.059 0 0 rpy=0 -1.5707963267948966 0

Commit message: Added top contact surface

File: urdf/robogami.urdf (robot description, URDF)
Before this commit: robot Robogami, 30 links, 29 joints
Links:
- added link topCenter
Joints:
- added joint topCenter: type fixed, parent top, child topCenter, origin xyz=-0.05629165124598851 0 0 rpy=0 3.141592653589793 0
