Commit message: Computing inertial properties from mesh geometry

File: urdf/robogami.urdf (robot description, URDF)
Before this commit: robot Robogami, 31 links, 30 joints
Links:
- link base: mass 0.01 -> 0.013721089544560527
- link leg1: mass 0.01 -> 0.0029841632454008504
- link leg1top: mass 0.01 -> 0.0029841632454008504
- link leg2: mass 0.01 -> 0.0029841632454008504
- link leg2top: mass 0.01 -> 0.0029841632454008504
- link leg3: mass 0.01 -> 0.0029841632454008504
- link leg3top: mass 0.01 -> 0.0029841632454008504
- link top: mass 0.01 -> 0.013721089544560527

Commit message: Adding point masses that represent motors

File: urdf/robogami.urdf (robot description, URDF)
Before this commit: robot Robogami, 31 links, 30 joints
Links:
- link base: mass 0.013721089544560527 -> 0.20872108954456053

File: urdf/robogami_custom.urdf (robot description, URDF)
Before this commit: robot Robogami, 31 links, 30 joints
Links:
- link base: mass 0.06495190518762683 -> 0.25995190518762684

Commit message: Make generated mesh file name config specific

File: urdf/robogami.urdf (robot description, URDF)
Before this commit: robot Robogami, 31 links, 30 joints
Links:
- link base: geometry visual mesh filename=package://robogami_description/meshes/robogami_base.stl
- link leg1: geometry visual mesh filename=package://robogami_description/meshes/robogami_leg.stl
- link leg1top: geometry visual mesh filename=package://robogami_description/meshes/robogami_leg.stl
- link leg2: geometry visual mesh filename=package://robogami_description/meshes/robogami_leg.stl
- link leg2top: geometry visual mesh filename=package://robogami_description/meshes/robogami_leg.stl
- link leg3: geometry visual mesh filename=package://robogami_description/meshes/robogami_leg.stl
- link leg3top: geometry visual mesh filename=package://robogami_description/meshes/robogami_leg.stl
- link top: geometry visual mesh filename=package://robogami_description/meshes/robogami_base.stl

File: urdf/robogami_custom.urdf (robot description, URDF)
Before this commit: robot Robogami, 31 links, 30 joints
Links:
- link base: geometry visual mesh filename=package://robogami_description/meshes/robogami_custom_base.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
- link leg1: geometry visual mesh filename=package://robogami_description/meshes/robogami_custom_leg.s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
- link leg1top: geometry visual mesh filename=package://robogami_description/meshes/robogami_custom_leg.s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
- link leg2: geometry visual mesh filename=package://robogami_description/meshes/robogami_custom_leg.s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
- link leg2top: geometry visual mesh filename=package://robogami_description/meshes/robogami_custom_leg.s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
- link leg3: geometry visual mesh filename=package://robogami_description/meshes/robogami_custom_leg.s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
- link leg3top: geometry visual mesh filename=package://robogami_description/meshes/robogami_custom_leg.s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
- link top: geometry visual mesh filename=package://robogami_description/meshes/robogami_custom_base.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

Commit message: Additional end-effector frame

File: urdf/robogami.urdf (robot description, URDF)
Before this commit: robot Robogami, 31 links, 30 joints
Links:
- added link endEffector
Joints:
- added joint ee: type fixed, parent topCenter, child endEffector, origin xyz=0 0 0 rpy=0 -1.5707963267948966 0

File: urdf/robogami_custom.urdf (robot description, URDF)
Before this commit: robot Robogami, 31 links, 30 joints
Links:
- added link endEffector
Joints:
- added joint ee: type fixed, parent topCenter, child endEffector, origin xyz=0 0 0 rpy=0 -1.5707963267948966 0

Commit message: Changed end-effector orientation frame orientation

File: urdf/robogami.urdf (robot description, URDF)
Before this commit: robot Robogami, 32 links, 31 joints
Joints:
- joint ee: origin xyz=0 0 0 rpy=0 -1.5707963267948966 0 -> xyz=0 0 0 rpy=3.141592653589793 -1.5707963267948966 0

File: urdf/robogami_custom.urdf (robot description, URDF)
Before this commit: robot Robogami, 32 links, 31 joints
Joints:
- joint ee: origin xyz=0 0 0 rpy=0 -1.5707963267948966 0 -> xyz=0 0 0 rpy=3.141592653589793 -1.5707963267948966 0
